File: Hardware/Control_Board/Control_Board.kicad_sch (KiCad schematic)
At the start: 1 part, among them IC2 ARD-NANO30NP

Commit message: Control board updates
Parts:
- removed IC2: ARD-NANO30NP, ARDNANO30NP, symbol Samacsys:ARD-NANO30NP
- added D1, D4: R_LED, symbol Device:LED
- added D2, D5: Y_LED, symbol Device:LED
- added D3, D6: G_LED, symbol Device:LED
- added J1: 825433-7, 8254337, symbol Samacsys:825433-7
Connections:
- new net GND: D1.1 (K), D2.1 (K), D3.1 (K), D4.1 (K), D5.1 (K), D6.1 (K), J1.7
- new net led1: D1.2 (A), J1.1
- new net led2: D2.2 (A), J1.2
- new net led3: D3.2 (A), J1.3
- new net led4: D4.2 (A), J1.4
- new net led5: D5.2 (A), J1.5
- new net led6: D6.2 (A), J1.6

Commit message: Sch rev 1 ready for review
Parts:
- removed D1, D4: R_LED, symbol Device:LED
- removed D2, D5: Y_LED, symbol Device:LED
- removed D3, D6: G_LED, symbol Device:LED
- removed J1: 825433-7, 8254337, symbol Samacsys:825433-7
- added A?: Arduino_Nano_v3.x, Module:Arduino_Nano, symbol MCU_Module:Arduino_Nano_v3.x
- added C? (x2): 22uF, Capacitor_SMD:C_1206_3216Metric, symbol OzoneController-rescue:C_Small-Device-OzoneController-rescue
- added C?: 100nF, Capacitor_SMD:C_0603_1608Metric, symbol OzoneController-rescue:C_Small-Device-OzoneController-rescue
- added C? (x2): 10uF, Capacitor_SMD:C_1206_3216Metric, symbol OzoneController-rescue:C_Small-Device-OzoneController-rescue
- added D? (x2): LED_Red_power, LED_SMD:LED_0603_1608Metric, symbol Device:LED_Small
- added J1: Raspberry_Pi_2_3, symbol Connector:Raspberry_Pi_2_3
- added J? (x4): Term_01x02, 1792863-2term_power:1792863, symbol Connector:Screw_Terminal_01x02
- added J? (x2): Screw_Terminal_01x02, TBL004-508-02BE-2GY:CUI_TBL004-508-02BE-2GY, symbol Connector:Screw_Terminal_01x02
- added K? (x4): ALQ3F12, ALQ3F12:ALQ3F12, symbol OzoneController-rescue:ALQ3F12-ALQ3F12-OzoneController-rescue
- added L?: 3.3uH, Inductor_SMD:L_10.4x10.4_H4.8, symbol OzoneController-rescue:L-Device-OzoneController-rescue
- added Q? (x2): Q_Dual_PMOS_S1G1S2G2D2D2D1D1, Package_SO:SOP-8_3.9x4.9mm_P1.27mm, symbol Device:Q_Dual_PMOS_S1G1S2G2D2D2D1D1
- added Q?: PMOS, Package_SO:SOIC-8_3.9x4.9mm_P1.27mm, symbol Project_Library:PMOS_AO4407A
- added R1: 10k, symbol Device:R_Small_US
- added R2: 20k, symbol Device:R_Small_US
- added R? (x2): 6.8k, Resistor_SMD:R_0402_1005Metric, symbol Device:R_Small_US
- added R?: 56.2k, Resistor_SMD:R_0402_1005Metric, symbol Device:R_Small_US
- added R? (x2): 10k, Resistor_SMD:R_0402_1005Metric, symbol Device:R_Small_US
- added U1, U2: ULN2003, Package_SO:SOIC-16_3.9x9.9mm_P1.27mm, symbol OzoneController-rescue:ULN2003-Transistor_Array-OzoneController-rescue
- added U?: TPS563200, Package_TO_SOT_SMD:SOT-23-6, symbol Regulator_Switching:TPS563200
Connections:
- net GND: now also A?.29 (GND), A?.4 (GND), C?.2, C?.2, C?.2, C?.2, J1.14 (GND), J1.20 (GND), J1.25 (GND), J1.30 (GND), J1.34 (GND), J1.39 (GND), J1.6 (GND), J1.9 (GND), J?.1 (Pin_1), J?.2 (Pin_2), Q?.2 (G), Q?.4, Q?.4 (G), R2.2, R?.1, R?.1, R?.1, R?.1, U1.8 (GND), U2.8 (GND), U?.1 (GND)
- new net: C?.1, L?.1, U?.2 (SW)
- new net: C?.1, C?.1, Q?.1 (D), Q?.2 (G), Q?.3 (eS), U?.3 (VIN), U?.5 (EN)
- new net: R?.1, R?.2, U?.4 (VFB)
- new net: C?.2, U?.6 (VBST)
- new net: J?.1 (Pin_1), J?.2 (Pin_2), K?.3 (NO) (x4)
- new net: D?.1 (K), R?.2, R?.2
- new net: C?.1, C?.1, L?.2, Q?.1 (S), R?.2
- new net: Q?.5 (D), Q?.7 (D)
- new net: Q?.6 (G), Q?.8 (G)
- new net: J1.10 (GPIO15/RXD), R1.1
- new net: D?.1 (K), R?.2
- new net +12V: D?.2 (A), J?.1 (Pin_1), J?.2 (Pin_2), Q?.5, Q?.6, Q?.7, Q?.8, U1.9 (COM), U2.9 (COM)
- new net +5V: A?.30 (VIN), D?.2 (A), J1.2 (5V), J1.4 (5V), Q?.3 (S)
- new net 120V_Hot: K?.4 (COM), K?.4 (COM), K?.4 (COM), K?.4 (COM)
- new net 12V: K?.1 (Coil), K?.1 (Coil), K?.1 (Coil), K?.1 (Coil)
- new net A0: A?.19 (A0)
- new net A1: A?.20 (A1)
- new net A2: A?.21 (A2)
- new net A4: A?.22 (A3)
- new net Pump1: U2.16 (O1)
- new net Pump2: U2.15 (O2)
- new net Pump3: U2.14 (O3)
- new net Pump4: U2.13 (O4)
- new net RX: A?.1 (D1/TX), R1.2, R2.1
- new net Relay1: K?.2 (Coil), U1.16 (O1)
- new net Relay2: K?.2 (Coil), U1.15 (O2)
- new net Relay3: K?.2 (Coil), K?.2 (Coil), U1.14 (O3)
- new net Relay4: U1.13 (O4)
- new net TX: A?.2 (D0/RX), J1.8 (GPIO14/TXD)
- new net U1/Pin1: J1.18 (GPIO24), U1.1 (I1)
- new net U1/Pin2: J1.22 (GPIO25), U1.2 (I2)
- new net U1/Pin3: J1.37 (GPIO26), U1.3 (I3)
- new net U1/Pin4: J1.13 (GPIO27), U1.4 (I4)
- new net U2/Pin1: J1.36 (GPIO16), U2.1 (I1)
- new net U2/Pin2: J1.11 (GPIO17), U2.2 (I2)
- new net U2/Pin3: J1.15 (GPIO22), U2.3 (I3)
- new net U2/Pin4: J1.16 (GPIO23), U2.4 (I4)
Other:
- note added: "12V Spare"
- note added: "12V to 5V SMPS Conversion"
- note added: "> From fused 120V-12VDC Converter"
- note added: "AC Earth 12V GND"
- note added: "Arduino Nano"
- note added: "Darlingtons"
- note added: "Fan"
- note added: "Heater"
- note added: "Input Power"
- note added: "Light 1"
- note added: "Light 2"
- note added: "Mains Control Relays"
- note added: "Protects as 12V/5V/3.3V loads (except relays) from reverse voltage and 5V SMPS from reverse current"
- note added: "Raspberry Pi"

Commit message: Control board layout
Parts:
- gave numbers to parts that had none: 27

Commit message: Control_Board updates
Parts:
- R1, R2: footprint (none) -> Resistor_SMD:R_0402_1005Metric_Pad0.72x0.64mm_HandSolder
Connections:
- net 12V is gone; now on net +12V: K1.1 (Coil), K2.1 (Coil), K3.1 (Coil), K4.1 (Coil)
- net A4: now also A1.23 (A4); no longer A1.22 (A3)
- new net A3: A1.22 (A3)
Changed lines of the file:
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@@
     (stroke (width 0) (type default) (color 0 0 0 0))
   )
-  (polyline (pts (xy 118.11 52.07) (xy 118.11 20.32))
+  (polyline (pts (xy 142.24 52.07) (xy 142.24 20.32))
     (stroke (width 0) (type default) (color 0 0 0 0))
   )
@@
     (stroke (width 0) (type default) (color 0 0 0 0))
   )
-  (polyline (pts (xy 118.11 52.07) (xy 167.64 52.07))
+  (polyline (pts (xy 142.24 52.07) (xy 167.64 52.07))
     (stroke (width 0) (type default) (color 0 0 0 0))
   )
@@
     (stroke (width 0) (type default) (color 0 0 0 0))
   )
-  (polyline (pts (xy 118.11 20.32) (xy 167.64 20.32))
+  (polyline (pts (xy 142.24 20.32) (xy 167.64 20.32))
     (stroke (width 0) (type default) (color 0 0 0 0))
   )
@@
     (effects (font (size 2.0066 2.0066)) (justify left bottom))
   )
-  (text "> From fused 120V-12VDC \n   Converter" (at 121.92 38.735 0)
+  (text "> From fused 120V-12VDC \n   Converter" (at 143.51 38.1 0)
     (effects (font (size 0.9906 0.9906)) (justify left bottom))
   )
@@
     (effects (font (size 2.0066 2.0066)) (justify left bottom))
   )
-  (text "Input Power" (at 134.62 19.05 0)
+  (text "Input Power" (at 146.05 19.05 0)
     (effects (font (size 2.0066 2.0066)) (justify left bottom))
   )
@@
     )
   )
-  (global_label "12V" (shape input) (at 246.38 64.77 180) (fields_autoplaced)
-    (effects (font (size 1.27 1.27)) (justify right))
-    (property "Intersheet References" "${INTERSHEET_REFS}" (id 0) (at 25.4 16.51 0)
-      (effects (font (size 1.27 1.27)) hide)
-    )
-  )
   (global_label "U1{slash}Pin2" (shape bidirectional) (at 46.99 154.94 180) (fields_autoplaced)
     (effects (font (size 1.27 1.27)) (justify right))
     (property "Intersheet References" "${INTERSHEET_REFS}" (id 0) (at 36.4731 154.8606 0)
       (effects (font (size 1.27 1.27)) (justify right) hide)
+    )
+  )
+  (global_label "A3" (shape bidirectional) (at 55.88 62.23 0) (fields_autoplaced)
+    (effects (font (size 1.27 1.27)) (justify left))
+    (property "Intersheet References" "${INTERSHEET_REFS}" (id 0) (at 60.5912 62.1506 0)
+      (effects (font (size 1.27 1.27)) (justify left) hide)
     )
   )
@@
     )
   )
-  (global_label "12V" (shape input) (at 246.38 121.92 180) (fields_autoplaced)
-    (effects (font (size 1.27 1.27)) (justify right))
-    (property "Intersheet References" "${INTERSHEET_REFS}" (id 0) (at 25.4 34.29 0)
-      (effects (font (size 1.27 1.27)) hide)
-    )
-  )
   (global_label "U2{slash}Pin1" (shape bidirectional) (at 46.99 127 180) (fields_autoplaced)
     (effects (font (size 1.27 1.27)) (justify right))
@@
     )
   )
-  (global_label "12V" (shape input) (at 246.38 85.09 180) (fields_autoplaced)
-    (effects (font (size 1.27 1.27)) (justify right))
-    (property "Intersheet References" "${INTERSHEET_REFS}" (id 0) (at 25.4 16.51 0)
-      (effects (font (size 1.27 1.27)) hide)
-    )
-  )
   (global_label "U1{slash}Pin3" (shape bidirectional) (at 114.3 120.65 180) (fields_autoplaced)
     (effects (font (size 1.27 1.27)) (justify right))
@@
     )
   )
-  (global_label "A4" (shape bidirectional) (at 55.88 62.23 0) (fields_autoplaced)
+  (global_label "A4" (shape bidirectional) (at 55.88 64.77 0) (fields_autoplaced)
     (effects (font (size 1.27 1.27)) (justify left))
-    (property "Intersheet References" "${INTERSHEET_REFS}" (id 0) (at 60.5912 62.1506 0)
+    (property "Intersheet References" "${INTERSHEET_REFS}" (id 0) (at 60.5912 64.6906 0)
       (effects (font (size 1.27 1.27)) (justify left) hide)
     )
@@
   (global_label "120V_Hot" (shape input) (at 259.08 101.6 0) (fields_autoplaced)
     (effects (font (size 1.27 1.27)) (justify left))
-    (property "Intersheet References" "${INTERSHEET_REFS}" (id 0) (at 25.4 16.51 0)
-      (effects (font (size 1.27 1.27)) hide)
-    )
-  )
-  (global_label "12V" (shape input) (at 246.38 104.14 180) (fields_autoplaced)
-    (effects (font (size 1.27 1.27)) (justify right))
     (property "Intersheet References" "${INTERSHEET_REFS}" (id 0) (at 25.4 16.51 0)
       (effects (font (size 1.27 1.27)) hide)
@@
       (effects (font (size 1.27 1.27)) (justify left))
     )
-    (property "Footprint" "" (id 2) (at 30.48 132.08 0)
+    (property "Footprint" "Resistor_SMD:R_0402_1005Metric_Pad0.72x0.64mm_HandSolder" (id 2) (at 30.48 132.08 0)
       (effects (font (size 1.27 1.27)) hide)
     )
@@
     (pin "7")
     (pin "8")
+    (pin "3")
+    (pin "4")
+    (pin "5")
+    (pin "6")
   )
   (symbol (lib_id "OzoneController-rescue:GND-power-OzoneController-rescue") (at 43.18 80.01 0) (mirror y) (unit 1)
@@
     )
     (property "Datasheet" "" (id 3) (at 134.62 149.86 0)
+      (effects (font (size 1.27 1.27)) hide)
+    )
+    (pin "1")
+  )
+  (symbol (lib_id "power:+12V") (at 246.38 64.77 0) (unit 1)
+    (in_bom yes) (on_board yes)
+    (property "Reference" "#PWR?" (id 0) (at 246.38 68.58 0)
+      (effects (font (size 1.27 1.27)) hide)
+    )
+    (property "Value" "+12V" (id 1) (at 246.761 60.3758 0))
+    (property "Footprint" "" (id 2) (at 246.38 64.77 0)
+      (effects (font (size 1.27 1.27)) hide)
+    )
+    (property "Datasheet" "" (id 3) (at 246.38 64.77 0)
       (effects (font (size 1.27 1.27)) hide)
     )
@@
       (effects (font (size 1.27 1.27)) (justify left))
     )
-    (property "Footprint" "" (id 2) (at 30.48 124.46 0)
+    (property "Footprint" "Resistor_SMD:R_0402_1005Metric_Pad0.72x0.64mm_HandSolder" (id 2) (at 30.48 124.46 0)
       (effects (font (size 1.27 1.27)) hide)
     )
@@
       (effects (font (size 1.27 1.27)) hide)
     )
+    (pin "1")
+    (pin "2")
+    (pin "7")
+    (pin "8")
     (pin "3")
     (pin "4")
@@
     (pin "2")
   )
+  (symbol (lib_id "power:+12V") (at 246.38 104.14 0) (unit 1)
+    (in_bom yes) (on_board yes)
+    (property "Reference" "#PWR?" (id 0) (at 246.38 107.95 0)
+      (effects (font (size 1.27 1.27)) hide)
+    )
+    (property "Value" "+12V" (id 1) (at 246.761 99.7458 0))
+    (property "Footprint" "" (id 2) (at 246.38 104.14 0)
+      (effects (font (size 1.27 1.27)) hide)
+    )
+    (property "Datasheet" "" (id 3) (at 246.38 104.14 0)
+      (effects (font (size 1.27 1.27)) hide)
+    )
+    (pin "1")
+  )
   (symbol (lib_id "OzoneController-rescue:ULN2003-Transistor_Array-OzoneController-rescue") (at 124.46 123.19 0) (unit 1)
     (in_bom yes) (on_board yes)
@@
     (pin "1")
   )
+  (symbol (lib_id "power:+12V") (at 246.38 121.92 0) (unit 1)
+    (in_bom yes) (on_board yes)
+    (property "Reference" "#PWR?" (id 0) (at 246.38 125.73 0)
+      (effects (font (size 1.27 1.27)) hide)
+    )
+    (property "Value" "+12V" (id 1) (at 246.761 117.5258 0))
+    (property "Footprint" "" (id 2) (at 246.38 121.92 0)
+      (effects (font (size 1.27 1.27)) hide)
+    )
+    (property "Datasheet" "" (id 3) (at 246.38 121.92 0)
+      (effects (font (size 1.27 1.27)) hide)
+    )
+    (pin "1")
+  )
   (symbol (lib_id "OzoneController-rescue:GND-power-OzoneController-rescue") (at 59.69 175.26 0) (unit 1)
     (in_bom yes) (on_board yes)
@@
     (pin "1")
     (pin "2")
+  )
+  (symbol (lib_id "power:+12V") (at 246.38 85.09 0) (unit 1)
+    (in_bom yes) (on_board yes)
+    (property "Reference" "#PWR?" (id 0) (at 246.38 88.9 0)
+      (effects (font (size 1.27 1.27)) hide)
+    )
+    (property "Value" "+12V" (id 1) (at 246.761 80.6958 0))
+    (property "Footprint" "" (id 2) (at 246.38 85.09 0)
+      (effects (font (size 1.27 1.27)) hide)
+    )
+    (property "Datasheet" "" (id 3) (at 246.38 85.09 0)
+      (effects (font (size 1.27 1.27)) hide)
+    )
+    (pin "1")
   )
   (symbol (lib_id "OzoneController-rescue:C_Small-Device-OzoneController-rescue") (at 189.865 36.83 0) (unit 1)
@@
       (reference "#PWR0123") (unit 1) (value "GND") (footprint "")
     )
+    (path "/624cfa7f-e026-43b9-a1c1-22606f3493f1"
+      (reference "#PWR?") (unit 1) (value "+12V") (footprint "")
+    )
+    (path "/bd8b64c4-3a32-4a60-a54b-7fb7edcc2728"
+      (reference "#PWR?") (unit 1) (value "+12V") (footprint "")
+    )
+    (path "/dac39aa9-78ac-4b87-a371-24e1b2ffb4c5"
+      (reference "#PWR?") (unit 1) (value "+12V") (footprint "")
+    )
+    (path "/f54d89ed-f3a0-4fef-a2fe-0800e2949686"
+      (reference "#PWR?") (unit 1) (value "+12V") (footprint "")
+    )
     (path "/69fa2526-fcef-486c-a5bb-ecb0750025e3"
       (reference "A1") (unit 1) (value "Arduino_Nano_v3.x") (footprint "Module:Arduino_Nano")
@@
     )
     (path "/7dc2f764-ab30-4f44-8435-ac3322d800ef"
-      (reference "R1") (unit 1) (value "10k") (footprint "")
+      (reference "R1") (unit 1) (value "10k") (footprint "Resistor_SMD:R_0402_1005Metric_Pad0.72x0.64mm_HandSolder")
     )
     (path "/0e71e6a2-5e60-4eee-95cf-83d155e51b78"
-      (reference "R2") (unit 1) (value "20k") (footprint "")
+      (reference "R2") (unit 1) (value "20k") (footprint "Resistor_SMD:R_0402_1005Metric_Pad0.72x0.64mm_HandSolder")
     )
     (path "/99183e99-67e4-4a75-9fa6-cc665606085f"
