File: Hardware/Control_Board/_autosave-Control_Board.kicad_sch (KiCad schematic)
At the start: 32 parts, among them J1 Raspberry_Pi_2_3, J2 Screw_Terminal_01x02, J3 Screw_Terminal_01x02, J4 Term_01x02, J5 Term_01x02, J6 Term_01x02, J7 Term_01x02, K1 ALQ3F12, K2 ALQ3F12, K3 ALQ3F12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

Commit message: Control_Board updates
Parts:
- J1: footprint (none) -> Library Loader:HDRV40W64P254_2X20_5080X500X884P
- R1, R2: footprint (none) -> Resistor_SMD:R_0402_1005Metric_Pad0.72x0.64mm_HandSolder
Connections:
- net 12V is gone; now on net +12V: K1.1 (Coil), K2.1 (Coil), K3.1 (Coil), K4.1 (Coil)
- net A4: now also A1.23 (A4); no longer A1.22 (A3)
- new net A3: A1.22 (A3)
Changed lines of the file:
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@@
     (stroke (width 0) (type default) (color 0 0 0 0))
   )
-  (polyline (pts (xy 140.97 52.07) (xy 140.97 20.32))
+  (polyline (pts (xy 142.24 52.07) (xy 142.24 20.32))
     (stroke (width 0) (type default) (color 0 0 0 0))
   )
@@
     (stroke (width 0) (type default) (color 0 0 0 0))
   )
-  (polyline (pts (xy 140.97 52.07) (xy 167.64 52.07))
+  (polyline (pts (xy 142.24 52.07) (xy 167.64 52.07))
     (stroke (width 0) (type default) (color 0 0 0 0))
   )
@@
     (stroke (width 0) (type default) (color 0 0 0 0))
   )
-  (polyline (pts (xy 140.97 20.32) (xy 167.64 20.32))
+  (polyline (pts (xy 142.24 20.32) (xy 167.64 20.32))
     (stroke (width 0) (type default) (color 0 0 0 0))
   )
@@
     (effects (font (size 2.0066 2.0066)) (justify left bottom))
   )
-  (text "Input Power" (at 144.78 19.05 0)
+  (text "Input Power" (at 146.05 19.05 0)
     (effects (font (size 2.0066 2.0066)) (justify left bottom))
   )
@@
     )
   )
-  (global_label "12V" (shape input) (at 246.38 64.77 180) (fields_autoplaced)
-    (effects (font (size 1.27 1.27)) (justify right))
-    (property "Intersheet References" "${INTERSHEET_REFS}" (id 0) (at 25.4 16.51 0)
-      (effects (font (size 1.27 1.27)) hide)
-    )
-  )
   (global_label "U1{slash}Pin2" (shape bidirectional) (at 46.99 154.94 180) (fields_autoplaced)
     (effects (font (size 1.27 1.27)) (justify right))
     (property "Intersheet References" "${INTERSHEET_REFS}" (id 0) (at 36.4731 154.8606 0)
       (effects (font (size 1.27 1.27)) (justify right) hide)
+    )
+  )
+  (global_label "A3" (shape bidirectional) (at 55.88 62.23 0) (fields_autoplaced)
+    (effects (font (size 1.27 1.27)) (justify left))
+    (property "Intersheet References" "${INTERSHEET_REFS}" (id 0) (at 60.5912 62.1506 0)
+      (effects (font (size 1.27 1.27)) (justify left) hide)
     )
   )
@@
     )
   )
-  (global_label "12V" (shape input) (at 246.38 121.92 180) (fields_autoplaced)
-    (effects (font (size 1.27 1.27)) (justify right))
-    (property "Intersheet References" "${INTERSHEET_REFS}" (id 0) (at 25.4 34.29 0)
-      (effects (font (size 1.27 1.27)) hide)
-    )
-  )
   (global_label "U2{slash}Pin1" (shape bidirectional) (at 46.99 127 180) (fields_autoplaced)
     (effects (font (size 1.27 1.27)) (justify right))
@@
     )
   )
-  (global_label "12V" (shape input) (at 246.38 85.09 180) (fields_autoplaced)
-    (effects (font (size 1.27 1.27)) (justify right))
-    (property "Intersheet References" "${INTERSHEET_REFS}" (id 0) (at 25.4 16.51 0)
-      (effects (font (size 1.27 1.27)) hide)
-    )
-  )
   (global_label "U1{slash}Pin3" (shape bidirectional) (at 114.3 120.65 180) (fields_autoplaced)
     (effects (font (size 1.27 1.27)) (justify right))
@@
     )
   )
-  (global_label "A4" (shape bidirectional) (at 55.88 62.23 0) (fields_autoplaced)
+  (global_label "A4" (shape bidirectional) (at 55.88 64.77 0) (fields_autoplaced)
     (effects (font (size 1.27 1.27)) (justify left))
-    (property "Intersheet References" "${INTERSHEET_REFS}" (id 0) (at 60.5912 62.1506 0)
+    (property "Intersheet References" "${INTERSHEET_REFS}" (id 0) (at 60.5912 64.6906 0)
       (effects (font (size 1.27 1.27)) (justify left) hide)
     )
@@
   (global_label "120V_Hot" (shape input) (at 259.08 101.6 0) (fields_autoplaced)
     (effects (font (size 1.27 1.27)) (justify left))
-    (property "Intersheet References" "${INTERSHEET_REFS}" (id 0) (at 25.4 16.51 0)
-      (effects (font (size 1.27 1.27)) hide)
-    )
-  )
-  (global_label "12V" (shape input) (at 246.38 104.14 180) (fields_autoplaced)
-    (effects (font (size 1.27 1.27)) (justify right))
     (property "Intersheet References" "${INTERSHEET_REFS}" (id 0) (at 25.4 16.51 0)
       (effects (font (size 1.27 1.27)) hide)
@@
       (effects (font (size 1.27 1.27)) (justify left))
     )
-    (property "Footprint" "" (id 2) (at 30.48 132.08 0)
+    (property "Footprint" "Resistor_SMD:R_0402_1005Metric_Pad0.72x0.64mm_HandSolder" (id 2) (at 30.48 132.08 0)
       (effects (font (size 1.27 1.27)) hide)
     )
@@
     )
     (property "Datasheet" "" (id 3) (at 134.62 149.86 0)
+      (effects (font (size 1.27 1.27)) hide)
+    )
+    (pin "1")
+  )
+  (symbol (lib_id "power:+12V") (at 246.38 64.77 0) (unit 1)
+    (in_bom yes) (on_board yes)
+    (property "Reference" "#PWR0124" (id 0) (at 246.38 68.58 0)
+      (effects (font (size 1.27 1.27)) hide)
+    )
+    (property "Value" "+12V" (id 1) (at 246.761 60.3758 0))
+    (property "Footprint" "" (id 2) (at 246.38 64.77 0)
+      (effects (font (size 1.27 1.27)) hide)
+    )
+    (property "Datasheet" "" (id 3) (at 246.38 64.77 0)
       (effects (font (size 1.27 1.27)) hide)
     )
@@
       (effects (font (size 1.27 1.27)) (justify left))
     )
-    (property "Footprint" "" (id 2) (at 30.48 124.46 0)
+    (property "Footprint" "Resistor_SMD:R_0402_1005Metric_Pad0.72x0.64mm_HandSolder" (id 2) (at 30.48 124.46 0)
       (effects (font (size 1.27 1.27)) hide)
     )
@@
     (pin "2")
   )
+  (symbol (lib_id "power:+12V") (at 246.38 104.14 0) (unit 1)
+    (in_bom yes) (on_board yes)
+    (property "Reference" "#PWR0126" (id 0) (at 246.38 107.95 0)
+      (effects (font (size 1.27 1.27)) hide)
+    )
+    (property "Value" "+12V" (id 1) (at 246.761 99.7458 0))
+    (property "Footprint" "" (id 2) (at 246.38 104.14 0)
+      (effects (font (size 1.27 1.27)) hide)
+    )
+    (property "Datasheet" "" (id 3) (at 246.38 104.14 0)
+      (effects (font (size 1.27 1.27)) hide)
+    )
+    (pin "1")
+  )
   (symbol (lib_id "OzoneController-rescue:ULN2003-Transistor_Array-OzoneController-rescue") (at 124.46 123.19 0) (unit 1)
     (in_bom yes) (on_board yes)
@@
     (pin "1")
   )
+  (symbol (lib_id "power:+12V") (at 246.38 121.92 0) (unit 1)
+    (in_bom yes) (on_board yes)
+    (property "Reference" "#PWR0127" (id 0) (at 246.38 125.73 0)
+      (effects (font (size 1.27 1.27)) hide)
+    )
+    (property "Value" "+12V" (id 1) (at 246.761 117.5258 0))
+    (property "Footprint" "" (id 2) (at 246.38 121.92 0)
+      (effects (font (size 1.27 1.27)) hide)
+    )
+    (property "Datasheet" "" (id 3) (at 246.38 121.92 0)
+      (effects (font (size 1.27 1.27)) hide)
+    )
+    (pin "1")
+  )
   (symbol (lib_id "OzoneController-rescue:GND-power-OzoneController-rescue") (at 59.69 175.26 0) (unit 1)
     (in_bom yes) (on_board yes)
@@
     (pin "2")
   )
+  (symbol (lib_id "power:+12V") (at 246.38 85.09 0) (unit 1)
+    (in_bom yes) (on_board yes)
+    (property "Reference" "#PWR0125" (id 0) (at 246.38 88.9 0)
+      (effects (font (size 1.27 1.27)) hide)
+    )
+    (property "Value" "+12V" (id 1) (at 246.761 80.6958 0))
+    (property "Footprint" "" (id 2) (at 246.38 85.09 0)
+      (effects (font (size 1.27 1.27)) hide)
+    )
+    (property "Datasheet" "" (id 3) (at 246.38 85.09 0)
+      (effects (font (size 1.27 1.27)) hide)
+    )
+    (pin "1")
+  )
   (symbol (lib_id "OzoneController-rescue:C_Small-Device-OzoneController-rescue") (at 189.865 36.83 0) (unit 1)
     (in_bom yes) (on_board yes)
@@
       (effects (font (size 1.27 1.27)) (justify left))
     )
-    (property "Footprint" "" (id 2) (at 67.31 142.24 0)
+    (property "Footprint" "Library Loader:HDRV40W64P254_2X20_5080X500X884P" (id 2) (at 67.31 142.24 0)
       (effects (font (size 1.27 1.27)) hide)
     )
@@
       (reference "#PWR0123") (unit 1) (value "GND") (footprint "")
     )
+    (path "/624cfa7f-e026-43b9-a1c1-22606f3493f1"
+      (reference "#PWR0124") (unit 1) (value "+12V") (footprint "")
+    )
+    (path "/f54d89ed-f3a0-4fef-a2fe-0800e2949686"
+      (reference "#PWR0125") (unit 1) (value "+12V") (footprint "")
+    )
+    (path "/bd8b64c4-3a32-4a60-a54b-7fb7edcc2728"
+      (reference "#PWR0126") (unit 1) (value "+12V") (footprint "")
+    )
+    (path "/dac39aa9-78ac-4b87-a371-24e1b2ffb4c5"
+      (reference "#PWR0127") (unit 1) (value "+12V") (footprint "")
+    )
     (path "/69fa2526-fcef-486c-a5bb-ecb0750025e3"
       (reference "A1") (unit 1) (value "Arduino_Nano_v3.x") (footprint "Module:Arduino_Nano")
@@
     )
     (path "/fe85cc68-8130-4bf2-9f13-5f4043caf601"
-      (reference "J1") (unit 1) (value "Raspberry_Pi_2_3") (footprint "")
+      (reference "J1") (unit 1) (value "Raspberry_Pi_2_3") (footprint "Library Loader:HDRV40W64P254_2X20_5080X500X884P")
     )
     (path "/bcb841d9-35e5-4c54-8b84-08cbcfa736af"
@@
     )
     (path "/7dc2f764-ab30-4f44-8435-ac3322d800ef"
-      (reference "R1") (unit 1) (value "10k") (footprint "")
+      (reference "R1") (unit 1) (value "10k") (footprint "Resistor_SMD:R_0402_1005Metric_Pad0.72x0.64mm_HandSolder")
     )
     (path "/0e71e6a2-5e60-4eee-95cf-83d155e51b78"
-      (reference "R2") (unit 1) (value "20k") (footprint "")
+      (reference "R2") (unit 1) (value "20k") (footprint "Resistor_SMD:R_0402_1005Metric_Pad0.72x0.64mm_HandSolder")
     )
     (path "/99183e99-67e4-4a75-9fa6-cc665606085f"
