File: Hardware/Control_Board/_autosave-Control_Board.kicad_sch (KiCad schematic)
At the start: 33 parts, among them J1 Raspberry_Pi_2_3, J2 Screw_Terminal_01x02, J3 Screw_Terminal_01x02, J4 19705-4301, J5 19705-4301, J6 19705-4301, J7 19705-4301, K1 ALQ3F12, K2 ALQ3F12, K3 ALQ3F12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

Commit message: v0.1 Ready for review
Parts:
- gave numbers to parts that had none: 1
- renumbered J7 to J112
Connections:
- net Relay3: no longer K4.5 (Coil)
- net Relay4: now also K4.5 (Coil)
Changed lines of the file:
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@@
     )
   )
-  (global_label "Relay3" (shape input) (at 246.38 129.54 180) (fields_autoplaced)
-    (effects (font (size 1.27 1.27)) (justify right))
-    (property "Intersheet References" "${INTERSHEET_REFS}" (id 0) (at 25.4 34.29 0)
-      (effects (font (size 1.27 1.27)) hide)
+  (global_label "Relay4" (shape input) (at 246.38 129.54 180) (fields_autoplaced)
+    (effects (font (size 1.27 1.27)) (justify right))
+    (property "Intersheet References" "${INTERSHEET_REFS}" (id 0) (at 237.6169 129.4606 0)
+      (effects (font (size 1.27 1.27)) (justify right) hide)
     )
   )
@@
   (symbol (lib_id "DGD:19705-4301") (at 251.46 152.4 90) (unit 1)
     (in_bom yes) (on_board yes) (fields_autoplaced)
-    (property "Reference" "J?" (id 0) (at 251.8953 136.4488 0)
+    (property "Reference" "J8" (id 0) (at 251.8953 136.4488 0)
       (effects (font (size 1.27 1.27)) (justify left) hide)
     )
@@
   (symbol (lib_id "DGD:19705-4301") (at 259.08 120.65 0) (unit 1)
     (in_bom yes) (on_board yes) (fields_autoplaced)
-    (property "Reference" "J7" (id 0) (at 275.0312 121.0853 0)
+    (property "Reference" "J112" (id 0) (at 275.0312 121.0853 0)
       (effects (font (size 1.27 1.27)) (justify left) hide)
     )
@@
       (reference "J6") (unit 1) (value "19705-4301") (footprint "197054301")
     )
+    (path "/0a00ce56-e043-4b74-9a27-cac43184ce2e"
+      (reference "J8") (unit 1) (value "19705-4301") (footprint "197054301")
+    )
     (path "/e56375de-4bd8-4884-8c56-e5e4bd2ccff8"
-      (reference "J7") (unit 1) (value "19705-4301") (footprint "197054301")
-    )
-    (path "/0a00ce56-e043-4b74-9a27-cac43184ce2e"
-      (reference "J?") (unit 1) (value "19705-4301") (footprint "197054301")
+      (reference "J112") (unit 1) (value "19705-4301") (footprint "197054301")
     )
     (path "/2f85830a-4c30-4fef-9111-0ef054c61d06"

Commit message: Vertical fix
Parts:
- J2, J3: footprint TBL004-508-02BE-2GY:CUI_TBL004-508-02BE-2GY -> Samacsys:197054301
Changed lines of the file:
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@@
       (effects (font (size 1.27 1.27)) hide)
     )
-    (property "Footprint" "TBL004-508-02BE-2GY:CUI_TBL004-508-02BE-2GY" (id 2) (at 152.4 31.75 0)
+    (property "Footprint" "Samacsys:197054301" (id 2) (at 152.4 31.75 0)
       (effects (font (size 1.27 1.27)) hide)
     )
@@
       (effects (font (size 1.27 1.27)) hide)
     )
-    (property "Footprint" "TBL004-508-02BE-2GY:CUI_TBL004-508-02BE-2GY" (id 2) (at 152.4 44.45 0)
+    (property "Footprint" "Samacsys:197054301" (id 2) (at 152.4 44.45 0)
       (effects (font (size 1.27 1.27)) hide)
     )
@@
     )
     (path "/bcb841d9-35e5-4c54-8b84-08cbcfa736af"
-      (reference "J2") (unit 1) (value "Screw_Terminal_01x02") (footprint "TBL004-508-02BE-2GY:CUI_TBL004-508-02BE-2GY")
+      (reference "J2") (unit 1) (value "Screw_Terminal_01x02") (footprint "Samacsys:197054301")
     )
     (path "/e54a720e-e37a-4304-9f41-3ff0b906ca43"
-      (reference "J3") (unit 1) (value "Screw_Terminal_01x02") (footprint "TBL004-508-02BE-2GY:CUI_TBL004-508-02BE-2GY")
+      (reference "J3") (unit 1) (value "Screw_Terminal_01x02") (footprint "Samacsys:197054301")
     )
     (path "/b4d9670f-2d45-4002-8536-d1693c21246b"
